File: Current Sense & overcurrent protection.sch (KiCad schematic (older format))
At the start: 32 parts, among them U6 TLV4316

Commit message: Changed some Diodes footprints to achieve the recommended ones on the datasheet
Parts:
- D20: value RSX201VA-30 -> RSX101VAM30TR
Changed lines of the file:
@@
 P 8100 9050
 F 0 "D20" H 8050 9130 50  0000 L CNN
-F 1 "RSX201VA-30" H 7820 8970 50  0000 L CNN
+F 1 "RSX101VAM30TR" H 7820 8970 50  0000 L CNN
 F 2 "Diodes_SMD:TUMD2" V 8100 9050 50  0001 C CNN
 F 3 "http://www.mouser.com/ds/2/348/ze-sbd_catalog-210813.pdf" V 8100 9050 50  0001 C CNN
