File: Test.sch (KiCad schematic (older format))
At the start: 88 parts, among them P1 CONN_01X02, P18 CONN_01X02, P19 CONN_01X02, P2 CONN_01X02, P24 CONN_01X02, P8 CONN_01X02, Q1 BSC440N10NS3GATMA1, Q2 BSC440N10NS3GATMA1, Q3 BSC440N10NS3GATMA1, Q4 BSC440N10NS3GATMA1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

Commit message: Changed some Diodes footprints to achieve the recommended ones on the datasheet
Parts:
- D50: footprint Diodes_SMD:DO-214AB -> Eigene Footprints:DO-214AA
Changed lines of the file:
@@
 F 0 "D50" H 1600 8100 50  0000 C CNN
 F 1 "TVS" H 1600 7800 50  0000 C CNN
-F 2 "Diodes_SMD:DO-214AB" H 1600 7950 50  0001 C CNN
+F 2 "Eigene Footprints:DO-214AA" H 1600 7950 50  0001 C CNN
 F 3 "http://www.mouser.com/ds/2/240/Littelfuse_TVS-Diode_SMBJ-48653.pdf" H 1600 7950 50  0001 C CNN
 	1    1600 7950
@@
 	8850 2550 9400 2550
 Connection ~ 3350 2550
-Connection ~ 2850 2250
 Connection ~ 3450 7750
 Connection ~ 3050 7550
